File: hardware/KungFuFlash.sch (KiCad schematic (older format))
At the start: 38 parts, among them J1 USB Power, J2 USB_B_Micro, J4 SWD, Q1 BC817, SW1 Reset, SW2 Menu, SW3 Special, U1 C64-Exp-Port, U2 AMS1117-3.3, U3 STM32F405RGTx, Y1 8MHz

Commit message: Long board cart PCB layout.
Parts:
- removed RN1, RN2: 100R, Resistor_SMD:R_Array_Convex_4x0603, symbol Device:R_Pack04
- added R10, R11, R12, R13, R14, R7, R8, R9: 100R, Resistor_SMD:R_0805_2012Metric_Pad1.15x1.40mm_HandSolder, symbol Device:R
- J2: value USB_B_Micro -> USB_B_Mini; footprint mod:Conn_USBmicro-B_ebay-side_TH -> Connector_USB:USB_Mini-B_Wuerth_65100516121_Horizontal
- SW1, SW2, SW3: footprint Button_Switch_THT:SW_PUSH_6mm_H8mm -> Button_Switch_THT:SW_Tactile_SPST_Angled_PTS645Vx83-2LFS
Changed lines of the file:
@@
 EESchema Schematic File Version 4
-LIBS:KungFuFlash-cache
 EELAYER 30 0
 EELAYER END
@@
 Sheet 1 1
 Title "Kung Fu Flash"
-Date "2019-12-14"
-Rev "1"
+Date "2021-03-18"
+Rev "2.1"
 Comp "open hardware"
 Comment1 ""
@@
 Wire Wire Line
 	2750 4000 2750 3650
-$Comp
-L Device:R_Pack04 RN1
-U 1 1 5DA66EB2
-P 1450 4550
-F 0 "RN1" V 1150 4550 50  0000 C CNN
-F 1 "100R" V 1650 4550 50  0000 C CNN
-F 2 "Resistor_SMD:R_Array_Convex_4x0603" V 1725 4550 50  0001 C CNN
-F 3 "~" H 1450 4550 50  0001 C CNN
-	1    1450 4550
-	0    1    1    0
-$EndComp
 Entry Wire Line
 	1000 4250 1100 4350
@@
 Entry Wire Line
 	1000 4550 1100 4650
-$Comp
-L Device:R_Pack04 RN2
-U 1 1 5DA6909D
-P 1450 5150
-F 0 "RN2" V 1150 5150 50  0000 C CNN
-F 1 "100R" V 1650 5150 50  0000 C CNN
-F 2 "Resistor_SMD:R_Array_Convex_4x0603" V 1725 5150 50  0001 C CNN
-F 3 "~" H 1450 5150 50  0001 C CNN
-	1    1450 5150
-	0    1    1    0
-$EndComp
 $Comp
 L power:GND #PWR0102
@@
 Wire Wire Line
 	1100 3550 1250 3550
-Wire Wire Line
-	1100 4350 1250 4350
-Wire Wire Line
-	1100 4450 1250 4450
-Wire Wire Line
-	1100 4550 1250 4550
-Wire Wire Line
-	1100 4650 1250 4650
-Wire Wire Line
-	1100 4950 1250 4950
-Wire Wire Line
-	1100 5050 1250 5050
-Wire Wire Line
-	1100 5150 1250 5150
-Wire Wire Line
-	1100 5250 1250 5250
-Wire Wire Line
-	1650 4350 1800 4350
-Wire Wire Line
-	1650 4450 1800 4450
-Wire Wire Line
-	1650 4550 1800 4550
-Wire Wire Line
-	1650 4650 1800 4650
-Wire Wire Line
-	1650 4950 1800 4950
-Wire Wire Line
-	1650 5050 1800 5050
-Wire Wire Line
-	1650 5150 1800 5150
-Wire Wire Line
-	1650 5250 1800 5250
 Wire Bus Line
 	900  5450 1900 5450
@@
 F 0 "SW2" H 8750 1550 50  0000 C CNN
 F 1 "Menu" H 8750 1250 50  0000 C CNN
-F 2 "Button_Switch_THT:SW_PUSH_6mm_H8mm" H 8750 1550 50  0001 C CNN
+F 2 "Button_Switch_THT:SW_Tactile_SPST_Angled_PTS645Vx83-2LFS" H 8750 1550 50  0001 C CNN
 F 3 "" H 8750 1550 50  0001 C CNN
 	1    8750 1350
@@
 F 0 "SW3" H 8750 2150 50  0000 C CNN
 F 1 "Special" H 8750 1850 50  0000 C CNN
-F 2 "Button_Switch_THT:SW_PUSH_6mm_H8mm" H 8750 2150 50  0001 C CNN
+F 2 "Button_Switch_THT:SW_Tactile_SPST_Angled_PTS645Vx83-2LFS" H 8750 2150 50  0001 C CNN
 F 3 "" H 8750 2150 50  0001 C CNN
 	1    8750 1950
@@
 P 9400 1650
 F 0 "J2" H 9400 2000 50  0000 C CNN
-F 1 "USB_B_Micro" H 9700 1300 50  0000 C CNN
-F 2 "mod:Conn_USBmicro-B_ebay-side_TH" H 9550 1600 50  0001 C CNN
+F 1 "USB_B_Mini" H 9700 1300 50  0000 C CNN
+F 2 "Connector_USB:USB_Mini-B_Wuerth_65100516121_Horizontal" H 9550 1600 50  0001 C CNN
 F 3 "~" H 9550 1600 50  0001 C CNN
 	1    9400 1650
@@
 F 0 "SW1" H 4200 1650 50  0000 C CNN
 F 1 "Reset" H 4200 1350 50  0000 C CNN
-F 2 "Button_Switch_THT:SW_PUSH_6mm_H8mm" H 4200 1650 50  0001 C CNN
+F 2 "Button_Switch_THT:SW_Tactile_SPST_Angled_PTS645Vx83-2LFS" H 4200 1650 50  0001 C CNN
 F 3 "" H 4200 1650 50  0001 C CNN
 	1    4200 1450
@@
 Wire Wire Line
 	8000 1950 8250 1950
+$Comp
+L Device:R R7
+U 1 1 605774A6
+P 1450 4350
+F 0 "R7" V 1450 4350 50  0000 C CNN
+F 1 "100R" V 1450 4950 50  0000 C CNN
+F 2 "Resistor_SMD:R_0805_2012Metric_Pad1.15x1.40mm_HandSolder" V 1380 4350 50  0001 C CNN
+F 3 "~" H 1450 4350 50  0001 C CNN
+	1    1450 4350
+	0    1    1    0
+$EndComp
+$Comp
+L Device:R R8
+U 1 1 60577C8A
+P 1450 4450
+F 0 "R8" V 1450 4450 50  0000 C CNN
+F 1 "100R" V 1450 5050 50  0000 C CNN
+F 2 "Resistor_SMD:R_0805_2012Metric_Pad1.15x1.40mm_HandSolder" V 1380 4450 50  0001 C CNN
+F 3 "~" H 1450 4450 50  0001 C CNN
+	1    1450 4450
+	0    1    1    0
+$EndComp
+$Comp
+L Device:R R9
+U 1 1 60577EB9
+P 1450 4550
+F 0 "R9" V 1450 4550 50  0000 C CNN
+F 1 "100R" V 1450 5150 50  0000 C CNN
+F 2 "Resistor_SMD:R_0805_2012Metric_Pad1.15x1.40mm_HandSolder" V 1380 4550 50  0001 C CNN
+F 3 "~" H 1450 4550 50  0001 C CNN
+	1    1450 4550
+	0    1    1    0
+$EndComp
+$Comp
+L Device:R R10
+U 1 1 605780ED
+P 1450 4650
+F 0 "R10" V 1450 4650 50  0000 C CNN
+F 1 "100R" V 1450 5250 50  0000 C CNN
+F 2 "Resistor_SMD:R_0805_2012Metric_Pad1.15x1.40mm_HandSolder" V 1380 4650 50  0001 C CNN
+F 3 "~" H 1450 4650 50  0001 C CNN
+	1    1450 4650
+	0    1    1    0
+$EndComp
+$Comp
+L Device:R R11
+U 1 1 6057FF63
+P 1450 4950
+F 0 "R11" V 1450 4950 50  0000 C CNN
+F 1 "100R" V 1450 5550 50  0000 C CNN
+F 2 "Resistor_SMD:R_0805_2012Metric_Pad1.15x1.40mm_HandSolder" V 1380 4950 50  0001 C CNN
+F 3 "~" H 1450 4950 50  0001 C CNN
+	1    1450 4950
+	0    1    1    0
+$EndComp
+$Comp
+L Device:R R12
+U 1 1 6057FF69
+P 1450 5050
+F 0 "R12" V 1450 5050 50  0000 C CNN
+F 1 "100R" V 1450 5650 50  0000 C CNN
+F 2 "Resistor_SMD:R_0805_2012Metric_Pad1.15x1.40mm_HandSolder" V 1380 5050 50  0001 C CNN
+F 3 "~" H 1450 5050 50  0001 C CNN
+	1    1450 5050
+	0    1    1    0
+$EndComp
+$Comp
+L Device:R R13
+U 1 1 6057FF6F
+P 1450 5150
+F 0 "R13" V 1450 5150 50  0000 C CNN
+F 1 "100R" V 1450 5750 50  0000 C CNN
+F 2 "Resistor_SMD:R_0805_2012Metric_Pad1.15x1.40mm_HandSolder" V 1380 5150 50  0001 C CNN
+F 3 "~" H 1450 5150 50  0001 C CNN
+	1    1450 5150
+	0    1    1    0
+$EndComp
+$Comp
+L Device:R R14
+U 1 1 6057FF75
+P 1450 5250
+F 0 "R14" V 1450 5250 50  0000 C CNN
+F 1 "100R" V 1450 5850 50  0000 C CNN
+F 2 "Resistor_SMD:R_0805_2012Metric_Pad1.15x1.40mm_HandSolder" V 1380 5250 50  0001 C CNN
+F 3 "~" H 1450 5250 50  0001 C CNN
+	1    1450 5250
+	0    1    1    0
+$EndComp
+Wire Wire Line
+	1100 4350 1300 4350
+Wire Wire Line
+	1100 4450 1300 4450
+Wire Wire Line
+	1100 4550 1300 4550
+Wire Wire Line
+	1100 4650 1300 4650
+Wire Wire Line
+	1600 4350 1800 4350
+Wire Wire Line
+	1600 4450 1800 4450
+Wire Wire Line
+	1600 4550 1800 4550
+Wire Wire Line
+	1600 4650 1800 4650
+Wire Wire Line
+	1100 4950 1300 4950
+Wire Wire Line
+	1100 5050 1300 5050
+Wire Wire Line
+	1100 5150 1300 5150
+Wire Wire Line
+	1100 5250 1300 5250
+Wire Wire Line
+	1600 5250 1800 5250
+Wire Wire Line
+	1600 5150 1800 5150
+Wire Wire Line
+	1600 4950 1800 4950
+Wire Wire Line
+	1600 5050 1800 5050
+Wire Wire Line
+	7250 2550 9950 2550
+Wire Wire Line
+	7250 1850 7800 1850
 Wire Wire Line
 	5450 3950 5850 3950
-Wire Wire Line
-	7250 2550 9950 2550
-Wire Wire Line
-	7250 1850 7800 1850
 Wire Bus Line
 	5350 3050 5350 4450
@@
 	1000 2950 1000 5150
 Wire Bus Line
+	7600 1550 7600 5450
+Wire Bus Line
 	3000 1750 3000 5450
-Wire Bus Line
-	7600 1550 7600 5450
 $EndSCHEMATC
